Commit message: Problems with Coag, Cam+, Cam- inputs
Former-commit-id: f8ccb63d0a3b33e40fe21b78bf63328411d2cfa5

File: dvrk_model/model/myDavinci.urdf (robot description, URDF)
Before this commit: robot dvrk_psm, 32 links, 31 joints
Links:
- added link one_tool_base_link
- added link one_tool_middle_link
- added link one_tool_tip_link
- added link two_tool_base_link
- added link two_tool_middle_link
- added link two_tool_tip_link
Joints:
- added joint one_fake_joint_1: type fixed, parent one_tool_wrist_sca_shaft_link, child one_tool_base_link, origin xyz=0 0 0 rpy=0 0 1.5708, limit lower=0.0 upper=3.1415 effort=1000.0 velocity=0.5
- added joint one_fake_joint_2: type fixed, parent one_tool_base_link, child one_tool_middle_link, origin xyz=0.00483 0 0 rpy=0 0 0, limit lower=0.0 upper=3.1415 effort=1000.0 velocity=0.5
- added joint one_fake_joint_3: type fixed, parent one_tool_middle_link, child one_tool_tip_link, origin xyz=0.00483 0 0 rpy=0 0 0, limit lower=0.0 upper=3.1415 effort=1000.0 velocity=0.5
- added joint two_fake_joint_1: type fixed, parent two_tool_wrist_sca_shaft_link, child two_tool_base_link, origin xyz=0 0 0 rpy=0 0 1.5708, limit lower=0.0 upper=3.1415 effort=1000.0 velocity=0.5
- added joint two_fake_joint_2: type fixed, parent two_tool_base_link, child two_tool_middle_link, origin xyz=0.00483 0 0 rpy=0 0 0, limit lower=0.0 upper=3.1415 effort=1000.0 velocity=0.5
- added joint two_fake_joint_3: type fixed, parent two_tool_middle_link, child two_tool_tip_link, origin xyz=0.00483 0 0 rpy=0 0 0, limit lower=0.0 upper=3.1415 effort=1000.0 velocity=0.5
- joint one_fixed_joint: origin xyz=-0.25 0.0 0.5 rpy=0.0 0.0 3.1415926 -> xyz=-0.015 -0.015 0.492 rpy=0.026 0.204 -2.927
- joint one_outer_wrist_open_angle_joint_2: mimic joint=one_outer_wrist_open_angle_joint_1 multiplier=-1 -> (none)
- joint two_outer_wrist_open_angle_joint_2: mimic joint=two_outer_wrist_open_angle_joint_1 multiplier=-1 -> (none)
